Commit message: Optimize robot model parameters and controller config
- Update base_link mass (0.87->4.0) and inertia for better simulation stability
- Replace simplified collision geometries with STL meshes for accuracy
- Fix left wheel joint orientation (rpy/axis) for correct mecanum motion
- Increase wheel joint effort (1.5->15.0) and damping/friction (0.01/0.1->0.3/0.3)
- Raise controller update rate from 50Hz to 200Hz
- Change cmd_vel relay QoS reliability from best_effort to reliable

File: src/M3Pro_robot_description/urdf/M3Pro.urdf.xacro (robot description, xacro)
@@ -20,13 +20,6 @@
         xyz="-0.0230945655800945 -0.000624366433481225 0.0924263074305092"
         rpy="0 0 0" />
-      <mass
-        value="0.870994544286568" />
-      <inertia
-        ixx="0.000924360334406296"
-        ixy="1.83790425775432E-06"
-        ixz="-6.57330050239333E-05"
-        iyy="0.000965356496722674"
-        iyz="4.19061203028733E-07"
-        izz="0.00166592475388463" />
+      <mass value="4.0" />
+      <inertia ixx="0.0097" ixy="0.0" ixz="0.0" iyy="0.0145" iyz="0.0" izz="0.0218" />
     </inertial>
     <visual>
@@ -84,5 +77,6 @@
       <origin xyz="0 0 0.016" rpy="0 0 0" />
       <geometry>
-        <box size="0.04 0.04 0.033"/>
+        <mesh
+          filename="package://M3Pro_robot_description/meshes/arm1.STL" />
       </geometry>
     </collision>
@@ -139,5 +133,6 @@
       <origin xyz="0 0 0.041" rpy="0 0 0" />
       <geometry>
-        <box size="0.035 0.04 0.083"/>
+        <mesh
+          filename="package://M3Pro_robot_description/meshes/arm2.STL" />
       </geometry>
     </collision>
@@ -194,5 +189,6 @@
       <origin xyz="0 0 0.041" rpy="0 0 0" />
       <geometry>
-        <box size="0.035 0.04 0.083"/>
+        <mesh
+          filename="package://M3Pro_robot_description/meshes/arm3.STL" />
       </geometry>
     </collision>
@@ -249,5 +245,6 @@
       <origin xyz="0 0 0.037" rpy="0 0 0" />
       <geometry>
-        <box size="0.05 0.04 0.075"/>
+        <mesh
+          filename="package://M3Pro_robot_description/meshes/arm4.STL" />
       </geometry>
     </collision>
@@ -304,5 +301,6 @@
       <origin xyz="0.01 0 0.03" rpy="0 0 0" />
       <geometry>
-        <box size="0.04 0.03 0.06"/>
+        <mesh
+          filename="package://M3Pro_robot_description/meshes/arm5.STL" />
       </geometry>
     </collision>
@@ -359,5 +357,6 @@
       <origin xyz="0.008 0 0" rpy="0 0 0" />
       <geometry>
-        <box size="0.03 0.008 0.004"/>
+        <mesh
+          filename="package://M3Pro_robot_description/meshes/rlink1.STL" />
       </geometry>
     </collision>
@@ -414,5 +413,6 @@
       <origin xyz="0.023 0.006 -0.005" rpy="0 0 0" />
       <geometry>
-        <box size="0.045 0.015 0.01"/>
+        <mesh
+          filename="package://M3Pro_robot_description/meshes/rlink2.STL" />
       </geometry>
     </collision>
@@ -468,5 +468,6 @@
       <origin xyz="0.009 0 0" rpy="0 0 0" />
       <geometry>
-        <box size="0.03 0.008 0.004"/>
+        <mesh
+          filename="package://M3Pro_robot_description/meshes/llink1.STL" />
       </geometry>
     </collision>
@@ -522,5 +523,6 @@
       <origin xyz="0.023 -0.006 -0.005" rpy="0 0 0" />
       <geometry>
-        <box size="0.045 0.015 0.01"/>
+        <mesh
+          filename="package://M3Pro_robot_description/meshes/llink2.STL" />
       </geometry>
     </collision>
@@ -576,5 +578,6 @@
       <origin xyz="0.015 0 -0.003" rpy="0 0 0" />
       <geometry>
-        <box size="0.03 0.004 0.006"/>
+        <mesh
+          filename="package://M3Pro_robot_description/meshes/rlink3.STL" />
       </geometry>
     </collision>
@@ -630,5 +633,6 @@
       <origin xyz="0.015 0 -0.003" rpy="0 0 0" />
       <geometry>
-        <box size="0.03 0.004 0.006"/>
+        <mesh
+          filename="package://M3Pro_robot_description/meshes/llink3.STL" />
       </geometry>
     </collision>
@@ -684,5 +688,6 @@
       <origin xyz="-0.065 0 -0.002" rpy="0 0 0" />
       <geometry>
-        <box size="0.13 0.015 0.006"/>
+        <mesh
+          filename="package://M3Pro_robot_description/meshes/Gripping.STL" />
       </geometry>
     </collision>
@@ -734,5 +739,6 @@
       <origin xyz="-0.001 -0.001 -0.002" rpy="0 0 0" />
       <geometry>
-        <box size="0.02 0.06 0.06"/>
+        <mesh
+          filename="package://M3Pro_robot_description/meshes/DCW2.STL" />
       </geometry>
     </collision>
@@ -784,5 +790,6 @@
       <origin xyz="-0.005 0.017 0" rpy="0 0 0" />
       <geometry>
-        <box size="0.025 0.09 0.025"/>
+        <mesh
+          filename="package://M3Pro_robot_description/meshes/Camera.STL" />
       </geometry>
     </collision>
@@ -1016,5 +1023,5 @@
     <origin
       xyz="0.0775753787975409 0.09775 0.0399999999999998"
-      rpy="-1.5707963267949 0 0" />
+      rpy="1.5707963267949 0 0" />
     <parent
       link="base_link" />
@@ -1022,9 +1029,7 @@
       link="lwheel1" />
     <axis
-      xyz="0 0 1" />
-    <limit
-      effort="1.5"
-      velocity="30.0" />
-    <dynamics damping="0.01" friction="0.1"/>
+      xyz="0 0 -1" />
+    <dynamics damping="0.3" friction="0.3" />
+    <limit effort="15.0" velocity="30.0" />
   </joint>
   <link
@@ -1070,5 +1075,5 @@
     <origin
       xyz="-0.0814246212024597 0.0977499999999995 0.0399976951545867"
-      rpy="-1.5707963267949 0 0" />
+      rpy="1.5707963267949 0 0" />
     <parent
       link="base_link" />
@@ -1076,9 +1081,7 @@
       link="lwheel2" />
     <axis
-      xyz="0 0 1" />
-    <limit
-      effort="1.5"
-      velocity="30.0" />
-    <dynamics damping="0.01" friction="0.1"/>
+      xyz="0 0 -1" />
+    <dynamics damping="0.3" friction="0.3" />
+    <limit effort="15.0" velocity="30.0" />
   </joint>
   <link
@@ -1131,8 +1134,6 @@
     <axis
       xyz="0 0 1" />
-    <limit
-      effort="1.5"
-      velocity="30.0" />
-    <dynamics damping="0.01" friction="0.1"/>
+    <dynamics damping="0.3" friction="0.3" />
+    <limit effort="15.0" velocity="30.0" />
   </joint>
   <link
@@ -1185,8 +1186,6 @@
     <axis
       xyz="0 0 1" />
-    <limit
-      effort="1.5"
-      velocity="30.0" />
-    <dynamics damping="0.01" friction="0.1"/>
+    <dynamics damping="0.3" friction="0.3" />
+    <limit effort="15.0" velocity="30.0" />
   </joint>
   <link

Commit message: feat: temporarily switch from mecanum to diff_drive controller for debugging
- Replace mecanum_drive_controller with diff_drive_controller (temporary)
- Add TODO comments for reverting back to mecanum drive later
- Reduce base_link collision box size for better stability
- Lower wheel joint damping (0.3->0.01) and friction (0.3->0.01)
- Reduce wheel effort (15->10) and velocity limits (30->20)
- Increase ground and wheel surface friction (mu 1.0->1.5)
- Simplify gripper link physics (remove unnecessary friction params)
- Add ground plane contact parameters (kp/kd) in world SDF
- Update cmd_vel relay topic to diff_drive_controller/cmd_vel_unstamped

File: src/M3Pro_robot_description/urdf/M3Pro.urdf.xacro (robot description, xacro)
@@ -38,7 +38,7 @@
     </visual>
     <collision>
-      <origin xyz="0 0 0.08" rpy="0 0 0" />
-      <geometry>
-        <box size="0.24 0.20 0.16"/>
+      <origin xyz="-0.02 0 0.05" rpy="0 0 0" />
+      <geometry>
+        <box size="0.2 0.16 0.06" />
       </geometry>
     </collision>
@@ -1030,6 +1030,6 @@
     <axis
       xyz="0 0 -1" />
-    <dynamics damping="0.3" friction="0.3" />
-    <limit effort="15.0" velocity="30.0" />
+    <dynamics damping="0.01" friction="0.01" />
+    <limit effort="10.0" velocity="20.0" />
   </joint>
   <link
@@ -1082,6 +1082,6 @@
     <axis
       xyz="0 0 -1" />
-    <dynamics damping="0.3" friction="0.3" />
-    <limit effort="15.0" velocity="30.0" />
+    <dynamics damping="0.01" friction="0.01" />
+    <limit effort="10.0" velocity="20.0" />
   </joint>
   <link
@@ -1134,6 +1134,6 @@
     <axis
       xyz="0 0 1" />
-    <dynamics damping="0.3" friction="0.3" />
-    <limit effort="15.0" velocity="30.0" />
+    <dynamics damping="0.01" friction="0.01" />
+    <limit effort="10.0" velocity="20.0" />
   </joint>
   <link
@@ -1186,6 +1186,6 @@
     <axis
       xyz="0 0 1" />
-    <dynamics damping="0.3" friction="0.3" />
-    <limit effort="15.0" velocity="30.0" />
+    <dynamics damping="0.01" friction="0.01" />
+    <limit effort="10.0" velocity="20.0" />
   </joint>
   <link

File: src/M3Pro_robot_description/urdf/M3Pro_robot_gazebo_materials.xacro (robot description, xacro)
@@ -9,11 +9,9 @@
     <gazebo reference="${ref}">
       <material>Gazebo/FlatBlack</material>
-      <mu1>1.0</mu1>
-      <mu2>1.0</mu2>
+      <mu1>1.5</mu1>
+      <mu2>1.5</mu2>
       <kp>1000000.0</kp>
-      <kd>100.0</kd>
+      <kd>10.0</kd>
       <minDepth>0.001</minDepth>
-      <maxVel>0.1</maxVel>
-      <fdir1>1 0 0</fdir1>
     </gazebo>
   </xacro:macro>
@@ -41,17 +39,7 @@
     <gazebo reference="rlink2">
       <material>Gazebo/White</material>
-      <self_collide>false</self_collide>
-      <mu1>100.0</mu1>
-      <mu2>100.0</mu2>
-      <kp>1000000.0</kp>
-      <kd>1.0</kd>
     </gazebo>
     <gazebo reference="llink2">
       <material>Gazebo/White</material>
-      <self_collide>false</self_collide>
-      <mu1>100.0</mu1>
-      <mu2>100.0</mu2>
-      <kp>1000000.0</kp>
-      <kd>1.0</kd>
     </gazebo>
     <xacro:wheel_friction ref="lwheel1" />

Commit message: comment out Camera link visual/collision to avoid duplicate with DCW2

File: src/M3Pro_robot_description/urdf/M3Pro.urdf.xacro (robot description, xacro)
@@ -773,4 +773,5 @@
         izz="5.78331989998345E-06" />
     </inertial>
+    <!-- visual/collision removed: avoid duplicate camera with DCW2 (depth_camera link)
     <visual>
       <origin
@@ -793,5 +794,5 @@
           filename="package://M3Pro_robot_description/meshes/Camera.STL" />
       </geometry>
-    </collision>
+    </collision> -->
   </link>
   <joint

Commit message: feat(description): update M3Pro material colors
Refine URDF and Gazebo material color definitions for visual consistency.

File: src/M3Pro_robot_description/urdf/M3Pro.urdf.xacro (robot description, xacro)
@@ -32,7 +32,7 @@
       </geometry>
       <material
-        name="">
-        <color
-          rgba="0.501960784313725 0.501960784313725 0.501960784313725 1" />
+        name="silver_grey">
+        <color
+          rgba="0.75 0.75 0.78 1" />
       </material>
     </visual>
@@ -69,7 +69,7 @@
       </geometry>
       <material
-        name="">
-        <color
-          rgba="0.776470588235294 0.756862745098039 0.737254901960784 1" />
+        name="orange">
+        <color
+          rgba="1.0 0.5 0.0 1" />
       </material>
     </visual>
@@ -125,7 +125,7 @@
       </geometry>
       <material
-        name="">
-        <color
-          rgba="0.898039215686275 0.917647058823529 0.929411764705882 1" />
+        name="white">
+        <color
+          rgba="0.95 0.95 0.95 1" />
       </material>
     </visual>
@@ -181,7 +181,7 @@
       </geometry>
       <material
-        name="">
-        <color
-          rgba="0.898039215686275 0.917647058823529 0.929411764705882 1" />
+        name="skyblue">
+        <color
+          rgba="0.3 0.7 1.0 1" />
       </material>
     </visual>
@@ -237,7 +237,7 @@
       </geometry>
       <material
-        name="">
-        <color
-          rgba="0.898039215686275 0.917647058823529 0.929411764705882 1" />
+        name="white">
+        <color
+          rgba="0.95 0.95 0.95 1" />
       </material>
     </visual>
@@ -293,7 +293,7 @@
       </geometry>
       <material
-        name="">
-        <color
-          rgba="0.203921568627451 0.203921568627451 0.203921568627451 1" />
+        name="orange">
+        <color
+          rgba="1.0 0.5 0.0 1" />
       </material>
     </visual>
@@ -349,7 +349,7 @@
       </geometry>
       <material
-        name="">
-        <color
-          rgba="0.898039215686275 0.917647058823529 0.929411764705882 1" />
+        name="yellow">
+        <color
+          rgba="1.0 0.9 0.0 1" />
       </material>
     </visual>
@@ -405,7 +405,7 @@
       </geometry>
       <material
-        name="">
-        <color
-          rgba="0.898039215686275 0.917647058823529 0.929411764705882 1" />
+        name="red">
+        <color
+          rgba="0.9 0.1 0.1 1" />
       </material>
     </visual>
@@ -460,7 +460,7 @@
       </geometry>
       <material
-        name="">
-        <color
-          rgba="0.898039215686275 0.917647058823529 0.929411764705882 1" />
+        name="yellow">
+        <color
+          rgba="1.0 0.9 0.0 1" />
       </material>
     </visual>
@@ -515,7 +515,7 @@
       </geometry>
       <material
-        name="">
-        <color
-          rgba="0.898039215686275 0.917647058823529 0.929411764705882 1" />
+        name="red">
+        <color
+          rgba="0.9 0.1 0.1 1" />
       </material>
     </visual>
@@ -570,7 +570,7 @@
       </geometry>
       <material
-        name="">
-        <color
-          rgba="0.898039215686275 0.917647058823529 0.929411764705882 1" />
+        name="yellow">
+        <color
+          rgba="1.0 0.9 0.0 1" />
       </material>
     </visual>
@@ -625,7 +625,7 @@
       </geometry>
       <material
-        name="">
-        <color
-          rgba="0.898039215686275 0.917647058823529 0.929411764705882 1" />
+        name="yellow">
+        <color
+          rgba="1.0 0.9 0.0 1" />
       </material>
     </visual>
@@ -680,7 +680,7 @@
       </geometry>
       <material
-        name="">
-        <color
-          rgba="0.898039215686275 0.917647058823529 0.929411764705882 1" />
+        name="yellow">
+        <color
+          rgba="1.0 0.9 0.0 1" />
       </material>
     </visual>
@@ -731,7 +731,7 @@
       </geometry>
       <material
-        name="">
-        <color
-          rgba="0.203921568627451 0.203921568627451 0.203921568627451 1" />
+        name="cyan_blue">
+        <color
+          rgba="0.0 0.6 1.0 1" />
       </material>
     </visual>
@@ -838,7 +838,7 @@
       </geometry>
       <material
-        name="">
-        <color
-          rgba="0.298039215686275 0.298039215686275 0.298039215686275 1" />
+        name="red">
+        <color
+          rgba="0.9 0.1 0.1 1" />
       </material>
     </visual>
@@ -894,7 +894,7 @@
       </geometry>
       <material
-        name="">
-        <color
-          rgba="0.298039215686275 0.298039215686275 0.298039215686275 1" />
+        name="lime_green">
+        <color
+          rgba="0.0 1.0 0.0 1" />
       </material>
     </visual>
@@ -950,7 +950,7 @@
       </geometry>
       <material
-        name="">
-        <color
-          rgba="0.298039215686275 0.298039215686275 0.298039215686275 1" />
+        name="purple">
+        <color
+          rgba="0.8 0.0 0.8 1" />
       </material>
     </visual>
@@ -1007,7 +1007,7 @@
       </geometry>
       <material
-        name="">
-        <color
-          rgba="0.298039215686275 0.298039215686275 0.298039215686275 1" />
+        name="black">
+        <color
+          rgba="0.1 0.1 0.1 1" />
       </material>
     </visual>
@@ -1059,7 +1059,7 @@
       </geometry>
       <material
-        name="">
-        <color
-          rgba="0.298039215686275 0.298039215686275 0.298039215686275 1" />
+        name="black">
+        <color
+          rgba="0.1 0.1 0.1 1" />
       </material>
     </visual>
@@ -1111,7 +1111,7 @@
       </geometry>
       <material
-        name="">
-        <color
-          rgba="0.298039215686275 0.298039215686275 0.298039215686275 1" />
+        name="black">
+        <color
+          rgba="0.1 0.1 0.1 1" />
       </material>
     </visual>
@@ -1163,7 +1163,7 @@
       </geometry>
       <material
-        name="">
-        <color
-          rgba="0.298039215686275 0.298039215686275 0.298039215686275 1" />
+        name="black">
+        <color
+          rgba="0.1 0.1 0.1 1" />
       </material>
     </visual>

File: src/M3Pro_robot_description/urdf/M3Pro_robot_gazebo_materials.xacro (robot description, xacro)
@@ -1,12 +1,24 @@
 <?xml version="1.0"?>
 <robot xmlns:xacro="http://www.ros.org/wiki/xacro">
-  <xacro:macro name="set_material" params="ref mat">
+  <xacro:macro name="gz_material" params="ref r g b a:=1.0">
     <gazebo reference="${ref}">
-      <material>${mat}</material>
+      <visual>
+        <material>
+          <ambient>${r} ${g} ${b} ${a}</ambient>
+          <diffuse>${r} ${g} ${b} ${a}</diffuse>
+          <specular>0.1 0.1 0.1 1</specular>
+        </material>
+      </visual>
     </gazebo>
   </xacro:macro>
   <xacro:macro name="wheel_friction" params="ref">
     <gazebo reference="${ref}">
-      <material>Gazebo/FlatBlack</material>
+      <visual>
+        <material>
+          <ambient>0.1 0.1 0.1 1</ambient>
+          <diffuse>0.1 0.1 0.1 1</diffuse>
+          <specular>0.05 0.05 0.05 1</specular>
+        </material>
+      </visual>
       <mu1>1.5</mu1>
       <mu2>1.5</mu2>
@@ -16,21 +28,30 @@
     </gazebo>
   </xacro:macro>
-  <xacro:macro name="gripper_link_props" params="ref mat:=Gazebo/White">
+  <xacro:macro name="gripper_link_props" params="ref r:=1.0 g:=0.9 b:=0.0">
     <gazebo reference="${ref}">
-      <material>${mat}</material>
+      <visual>
+        <material>
+          <ambient>${r} ${g} ${b} 1</ambient>
+          <diffuse>${r} ${g} ${b} 1</diffuse>
+          <specular>0.1 0.1 0.1 1</specular>
+        </material>
+      </visual>
       <self_collide>false</self_collide>
     </gazebo>
   </xacro:macro>
   <xacro:macro name="gazebo_materials">
-    <xacro:set_material ref="base_link"       mat="Gazebo/Grey" />
-    <xacro:set_material ref="arm_base_Link"   mat="Gazebo/Green" />
-    <xacro:set_material ref="arm1"            mat="Gazebo/White" />
-    <xacro:set_material ref="arm2"            mat="Gazebo/White" />
-    <xacro:set_material ref="arm3"            mat="Gazebo/White" />
-    <xacro:set_material ref="arm4"            mat="Gazebo/White" />
-    <xacro:set_material ref="arm5"            mat="Gazebo/DarkGrey" />
-    <xacro:set_material ref="Gripping"        mat="Gazebo/White" />
-    <xacro:set_material ref="DCW2"            mat="Gazebo/DarkGrey" />
-    <xacro:set_material ref="Camera"          mat="Gazebo/Grey" />
+    <xacro:gz_material ref="base_link"       r="0.75" g="0.75" b="0.78" />
+    <xacro:gz_material ref="arm_base_Link"   r="0.0" g="0.63" b="0.24" />
+    <xacro:gz_material ref="arm1"            r="1.0" g="0.5" b="0.0" />
+    <xacro:gz_material ref="arm2"            r="0.95" g="0.95" b="0.95" />
+    <xacro:gz_material ref="arm3"            r="0.3" g="0.7" b="1.0" />
+    <xacro:gz_material ref="arm4"            r="0.95" g="0.95" b="0.95" />
+    <xacro:gz_material ref="arm5"            r="1.0" g="0.5" b="0.0" />
+    <xacro:gz_material ref="Gripping"        r="1.0" g="0.9" b="0.0" />
+    <xacro:gz_material ref="DCW2"            r="0.0" g="0.6" b="1.0" />
+    <xacro:gz_material ref="Camera"          r="0.15" g="0.15" b="0.15" />
+    <xacro:gz_material ref="imu_frame"       r="0.9" g="0.1" b="0.1" />
+    <xacro:gz_material ref="laser0_frame"    r="0.0" g="1.0" b="0.0" />
+    <xacro:gz_material ref="laser1_frame"    r="0.8" g="0.0" b="0.8" />
     <xacro:gripper_link_props ref="rlink1" />
     <xacro:gripper_link_props ref="llink1" />
@@ -38,5 +59,11 @@
     <xacro:gripper_link_props ref="llink3" />
     <gazebo reference="rlink2">
-      <material>Gazebo/White</material>
+      <visual>
+        <material>
+          <ambient>0.9 0.1 0.1 1</ambient>
+          <diffuse>0.9 0.1 0.1 1</diffuse>
+          <specular>0.1 0.1 0.1 1</specular>
+        </material>
+      </visual>
       <self_collide>false</self_collide>
       <mu1>100.0</mu1>
@@ -46,5 +73,11 @@
     </gazebo>
     <gazebo reference="llink2">
-      <material>Gazebo/White</material>
+      <visual>
+        <material>
+          <ambient>0.9 0.1 0.1 1</ambient>
+          <diffuse>0.9 0.1 0.1 1</diffuse>
+          <specular>0.1 0.1 0.1 1</specular>
+        </material>
+      </visual>
       <self_collide>false</self_collide>
       <mu1>100.0</mu1>
